Commit message: Созданы файлы URDF

File: description/robot_core.xacro (robot description, xacro)
@@ -21,5 +21,5 @@
         <parent link="base_link"/>
         <child link="chassis"/>
-        <origin xyz="-0.15 0 0"/>
+        <origin xyz="-0.30 0 0"/>
     </joint>
     <link name="chassis">
@@ -42,5 +42,5 @@
         </xacro:inertial_box>
     </link>
-    <!-- LEFT WHEEL LINK -->
+    <!--LEFT WHEEL LINK -->
     <joint name="left_wheel_joint" type="continuous">
         <parent link="base_link"/>
@@ -70,5 +70,5 @@
         <parent link="base_link"/>
         <child link="right_wheel"/>
-        <origin xyz="0 -0.175 0.016" rpy="-${pi/2} 0 0" />
+        <origin xyz="0 -0.175 0.016" rpy="${pi/2} 0 0" />
         <axis xyz="0 0 -1"/>
     </joint>
@@ -94,5 +94,5 @@
         <parent link="chassis"/>
         <child link="left_caster_wheel"/>
-        <origin xyz="0.30 0.1 0"/>
+        <origin xyz="0.15 0.1 0"/>
     </joint>
     <link name="left_caster_wheel">
@@ -117,5 +117,5 @@
         <parent link="chassis"/>
         <child link="right_caster_wheel"/>
-        <origin xyz="0.30 -0.1 0"/>
+        <origin xyz="0.15 -0.1 0"/>
     </joint>
     <link name="right_caster_wheel">
